File: cad/D1Mini_Wuerfel_aktuell.kicad_pcb (KiCad board)
At the start: 2 copper layers, 64 x 115 mm, 44 parts, among them K1 1x03, T1 IRF9952, T2 FDN337N, T3 IRLML9301, U1 WeMos_D1_mini, U2 TSR1-2450

Commit message: readme proofreading
Parts:
- added R1_SMT1: 100K, Resistor_SMD:R_1206_3216Metric, F.Cu at (110.3, 138.0)
- moved R1_THT1 23.9 mm to (110.2, 138.0)
- moved BAT1 6.70 mm to (105.2, 141.0)
- moved D27 1.12 mm to (143.5, 144.0)
- moved T2 0.25 mm to (117.8, 134.5)
- renumbered R1 to R1_THT1
Connections:
- S1 pad 3: GND -> (no net)
- S2 pad 3: GND -> (no net)
- S3 pad 3: GND -> (no net)
Routing:
- net XFET: track 0.00 -> 54.0 mm, vias 0 -> 2
- net +9V: track 0.00 -> 39.9 mm
- net U2_VIN: track 21.7 -> 45.5 mm
- net D1: track 0.00 -> 22.9 mm, vias 0 -> 2
- net GND: track 0.00 -> 11.5 mm, vias 0 -> 2
- net Net-(D27-Pad2): track 91.6 -> 92.5 mm
- added copper zone on F.Cu, net GND

Commit message: updated cad
Parts:
- moved R1_SMT1 0.84 mm to (110.3, 137.2)
- moved R1_THT1 0.84 mm to (110.2, 137.2)
Changed lines of the file:
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@@
       (outputformat 1)
       (mirror false)
-      (drillshape 1)
+      (drillshape 0)
       (scaleselection 1)
-      (outputdirectory "")
+      (outputdirectory "gerber/")
     )
   )
@@
   )
   (footprint "Resistor_SMD:R_1206_3216Metric" (layer "F.Cu")
-    (at 110.2875 138)
+    (at 110.2875 137.16)
     (descr "Resistor SMD 1206 (3216 Metric), square (rectangular) end terminal, IPC_7351 nominal, (Body size source: IPC-SM-782 page 72, https://www.pcb-3d.com/wordpress/wp-content/uploads/ipc-sm-782a_amendment_1_and_2.pdf), generated with kicad-footprint-generator")
     (tags "resistor")
@@
         (effects (font (size 1 1) (thickness 0.15)))
     )
-    (fp_text value "100K" (at 0 1.82) (layer "F.Fab")
+    (fp_text value "100K" (at 2.1837 -2.0338) (layer "F.Fab")
         (effects (font (size 1 1) (thickness 0.15)))
     )
@@
     (fp_line (start 1.6 0.8) (end -1.6 0.8)
       (stroke (width 0.1) (type solid)) (layer "F.Fab"))
-    (pad "1" smd roundrect (at -1.4625 0) (size 1.125 1.75) (layers "F.Cu" "F.Paste" "F.Mask") (roundrect_rratio 0.222222)
+    (pad "1" smd roundrect (at -1.4625 0) (size 1.125 1.75) (layers "F.Cu" "F.Paste" "F.Mask") (roundrect_rratio 0.2222222222)
       (net 2 "+9V") (pintype "passive"))
-    (pad "2" smd roundrect (at 1.4625 0) (size 1.125 1.75) (layers "F.Cu" "F.Paste" "F.Mask") (roundrect_rratio 0.222222)
+    (pad "2" smd roundrect (at 1.4625 0) (size 1.125 1.75) (layers "F.Cu" "F.Paste" "F.Mask") (roundrect_rratio 0.2222222222)
       (net 31 "XFET") (pintype "passive"))
     (model "${KICAD6_3DMODEL_DIR}/Resistor_SMD.3dshapes/R_1206_3216Metric.wrl"
@@
   )
   (footprint "D1Mini_Wuerfel_aktuell:0207_37" placed (layer "B.Cu")
-    (at 110.25 138)
+    (at 110.25 137.16)
     (property "Sheetfile" "D1Mini_Wuerfel_aktuell.kicad_sch")
     (property "Sheetname" "")
@@
   (segment (start 116.1 146.3) (end 117.95 144.45) (width 0.7) (layer "F.Cu") (net 2))
   (segment (start 107.97 146.3) (end 116.1 146.3) (width 0.7) (layer "F.Cu") (net 2))
-  (segment (start 105.17 138) (end 108.825 138) (width 0.3) (layer "F.Cu") (net 2))
+  (segment (start 105.17 137.16) (end 108.825 137.16) (width 0.3) (layer "F.Cu") (net 2))
   (segment (start 105.17 143.5) (end 105.25 143.58) (width 0.7) (layer "F.Cu") (net 2))
   (segment (start 105.25 143.58) (end 107.97 146.3) (width 0.7) (layer "F.Cu") (net 2))
@@
   (segment (start 138.94 131.44) (end 138.94 135.25) (width 1) (layer "F.Cu") (net 30))
   (segment (start 126.115 133.8) (end 126.115 132.37) (width 0.3) (layer "F.Cu") (net 31))
-  (segment (start 111.75 138) (end 115.33 138) (width 0.3) (layer "F.Cu") (net 31))
+  (segment (start 115.33 137.16) (end 115.33 137.46) (width 0.3) (layer "F.Cu") (net 31))
+  (segment (start 111.75 137.16) (end 115.33 137.16) (width 0.3) (layer "F.Cu") (net 31))
   (segment (start 129.95 139.2) (end 128.655 139.2) (width 0.3) (layer "F.Cu") (net 31))
-  (segment (start 117.95 142.55) (end 117.95 140.62) (width 0.3) (layer "F.Cu") (net 31))
-  (segment (start 117.68 135.65) (end 115.33 138) (width 0.3) (layer "F.Cu") (net 31))
+  (segment (start 117.08 135.65) (end 115.57 137.16) (width 0.3) (layer "F.Cu") (net 31))
   (segment (start 138.42 144) (end 134.75 144) (width 0.3) (layer "F.Cu") (net 31))
-  (segment (start 117.95 140.62) (end 115.33 138) (width 0.3) (layer "F.Cu") (net 31))
   (segment (start 117.75 135.65) (end 118.15 135.25) (width 0.3) (layer "F.Cu") (net 31))
+  (segment (start 115.33 137.46) (end 117.95 140.08) (width 0.3) (layer "F.Cu") (net 31))
   (segment (start 124 135.25) (end 124.845 134.405) (width 0.3) (layer "F.Cu") (net 31))
   (segment (start 134.75 144) (end 129.95 139.2) (width 0.3) (layer "F.Cu") (net 31))
-  (segment (start 117.75 135.65) (end 117.68 135.65) (width 0.3) (layer "F.Cu") (net 31))
+  (segment (start 117.95 140.08) (end 117.95 142.55) (width 0.3) (layer "F.Cu") (net 31))
   (segment (start 124.845 134.405) (end 124.845 133.8) (width 0.3) (layer "F.Cu") (net 31))
   (segment (start 131.25 132) (end 134.75 135.5) (width 0.3) (layer "F.Cu") (net 31))
+  (segment (start 117.75 135.65) (end 117.08 135.65) (width 0.3) (layer "F.Cu") (net 31))
   (segment (start 124.845 133.8) (end 126.115 133.8) (width 0.3) (layer "F.Cu") (net 31))
+  (segment (start 115.57 137.16) (end 115.33 137.16) (width 0.3) (layer "F.Cu") (net 31))
   (segment (start 126.485 132) (end 131.25 132) (width 0.3) (layer "F.Cu") (net 31))
   (segment (start 126.115 132.37) (end 126.485 132) (width 0.3) (layer "F.Cu") (net 31))
