File: cad/D1Mini_Wuerfel_aktuell.kicad_sch (KiCad schematic)
At the start: 41 parts, among them K1 1x03, T1 IRF9952, T2 FDN337N, T3 IRLML9301, U1 WeMos_D1_mini, U2 TSR1-2450

Commit message: updated cad
Other:
- moved on the sheet: K1
Changed lines of the file:
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@@
     (stroke (width 0) (type default))
   )
-  (wire (pts (xy 269.24 122.555) (xy 274.32 127.635))
+  (wire (pts (xy 268.5034 122.5804) (xy 273.5834 127.6604))
     (stroke (width 0) (type default))
   )
@@
     (stroke (width 0) (type default))
   )
+  (wire (pts (xy 268.5288 122.555) (xy 267.97 122.555))
+    (stroke (width 0) (type default))
+  )
   (wire (pts (xy 187.96 59.055) (xy 186.69 59.055))
     (stroke (width 0) (type default))
@@
     (stroke (width 0) (type default))
   )
+  (wire (pts (xy 268.5288 122.5804) (xy 268.5288 122.555))
+    (stroke (width 0) (type default))
+  )
   (wire (pts (xy 171.45 92.075) (xy 171.45 93.345))
     (stroke (width 0) (type default))
@@
     (stroke (width 0) (type default))
   )
-  (wire (pts (xy 274.32 127.635) (xy 279.4 127.635))
+  (wire (pts (xy 273.5834 127.6604) (xy 276.225 127.6604))
     (stroke (width 0) (type default))
   )
@@
     (stroke (width 0) (type default))
   )
-  (wire (pts (xy 269.24 122.555) (xy 267.97 122.555))
+  (wire (pts (xy 268.5034 122.5804) (xy 268.5288 122.5804))
     (stroke (width 0) (type default))
   )
@@
     (stroke (width 0) (type default))
   )
-  (wire (pts (xy 279.4 121.285) (xy 279.4 125.095))
+  (wire (pts (xy 276.225 121.3104) (xy 276.225 125.1204))
     (stroke (width 0) (type default))
   )
@@
     (stroke (width 0) (type default))
   )
-  (wire (pts (xy 279.4 130.175) (xy 279.4 133.985))
+  (wire (pts (xy 276.225 130.2004) (xy 276.225 134.0104))
     (stroke (width 0) (type default))
   )
@@
     )
   )
-  (symbol (lib_id "D1Mini_Wuerfel_aktuell-eagle-import:K1X03_BUCHSE_8") (at 279.4 127.635 90) (mirror x) (unit 1)
-    (in_bom yes) (on_board yes) (dnp no) (fields_autoplaced)
-    (property "Reference" "K1" (at 281.94 126.365 90)
+  (symbol (lib_id "D1Mini_Wuerfel_aktuell-eagle-import:K1X03_BUCHSE_8") (at 276.225 127.6604 90) (mirror x) (unit 1)
+    (in_bom yes) (on_board yes) (dnp no)
+    (property "Reference" "K1" (at 278.0792 126.365 90)
       (effects (font (size 2 1.7)) (justify right))
     )
-    (property "Value" "1x03" (at 281.94 128.905 90)
+    (property "Value" "1x03" (at 278.0792 128.9812 90)
       (effects (font (size 2 1.7)) (justify right))
     )
-    (property "Footprint" "D1Mini_Wuerfel_aktuell:1X03_BUCHSE_8" (at 279.4 127.635 0)
-      (effects (font (size 1.27 1.27)) hide)
-    )
-    (property "Datasheet" "" (at 279.4 127.635 0)
+    (property "Footprint" "D1Mini_Wuerfel_aktuell:1X03_BUCHSE_8" (at 276.225 127.6604 0)
+      (effects (font (size 1.27 1.27)) hide)
+    )
+    (property "Datasheet" "" (at 276.225 127.6604 0)
       (effects (font (size 1.27 1.27)) hide)
     )
@@
     )
   )
-  (symbol (lib_id "power:GND") (at 279.4 133.985 0) (unit 1)
-    (in_bom yes) (on_board yes) (dnp no) (fields_autoplaced)
-    (property "Reference" "#PWR053" (at 279.4 140.335 0)
-      (effects (font (size 1.27 1.27)) hide)
-    )
-    (property "Value" "GND" (at 279.4 139.065 0)
-      (effects (font (size 1.27 1.27)))
-    )
-    (property "Footprint" "" (at 279.4 133.985 0)
-      (effects (font (size 1.27 1.27)) hide)
-    )
-    (property "Datasheet" "" (at 279.4 133.985 0)
+  (symbol (lib_id "power:GND") (at 276.225 134.0104 0) (unit 1)
+    (in_bom yes) (on_board yes) (dnp no) (fields_autoplaced)
+    (property "Reference" "#PWR053" (at 276.225 140.3604 0)
+      (effects (font (size 1.27 1.27)) hide)
+    )
+    (property "Value" "GND" (at 276.225 139.0904 0)
+      (effects (font (size 1.27 1.27)))
+    )
+    (property "Footprint" "" (at 276.225 134.0104 0)
+      (effects (font (size 1.27 1.27)) hide)
+    )
+    (property "Datasheet" "" (at 276.225 134.0104 0)
       (effects (font (size 1.27 1.27)) hide)
     )
@@
     )
   )
-  (symbol (lib_id "power:+5V") (at 279.4 121.285 0) (unit 1)
-    (in_bom yes) (on_board yes) (dnp no) (fields_autoplaced)
-    (property "Reference" "#PWR054" (at 279.4 125.095 0)
-      (effects (font (size 1.27 1.27)) hide)
-    )
-    (property "Value" "+5V" (at 279.4 116.205 0)
-      (effects (font (size 1.27 1.27)))
-    )
-    (property "Footprint" "" (at 279.4 121.285 0)
-      (effects (font (size 1.27 1.27)) hide)
-    )
-    (property "Datasheet" "" (at 279.4 121.285 0)
-      (effects (font (size 1.27 1.27)) hide)
-    )
+  (symbol (lib_id "power:+5V") (at 276.225 121.3104 0) (unit 1)
+    (in_bom yes) (on_board yes) (dnp no) (fields_autoplaced)
+    (property "Reference" "#PWR054" (at 276.225 125.1204 0)
+      (effects (font (size 1.27 1.27)) hide)
+    )
+    (property "Value" "+5V" (at 276.225 116.2304 0)
+      (effects (font (size 1.27 1.27)))
+    )
+    (property "Footprint" "" (at 276.225 121.3104 0)
+      (effects (font (size 1.27 1.27)) hide)
+    )
+    (property "Datasheet" "" (at 276.225 121.3104 0)
+      (effects (font (size 1.27 1.27)) hide)
+    )
